Commit message: trying to make things work

File: urdf/ur10e_with_robotiq_gripper.urdf.xacro (robot description, xacro)
@@ -1,4 +1,4 @@
 <?xml version="1.0"?>
-<robot xmlns:xacro="http://wiki.ros.org/xacro" name="brrrrr">
+<robot xmlns:xacro="http://wiki.ros.org/xacro" name="ur10e_with_eef">
   <!-- include macros for ur10e and the end effector (eef) model -->
   <xacro:include filename="$(find robotiq_85_description)/urdf/robotiq_85_gripper_macro.urdf.xacro" />
@@ -11,15 +11,8 @@
         <origin xyz="0 0 0" rpy="0 0 0"/>
     </xacro:robotiq_85_gripper>
-    <!-- attach eef to ur10e model -->
-    <!-- Note: this assumes that the 'my_eef' macro defines a 'base_link'
-         link which is the start of it's kinematic chain (if any) -->
-    <!-- <joint name="${prefix}robot_flange-${prefix}eef_base_link" type="fixed">
-      <origin xyz="0 0 0" rpy="0 0 0" />
-      <parent link="${prefix}robot_flange" />
-      <child link="${prefix}eef_base_link" />
-    </joint> -->
   </xacro:macro>
   <xacro:ur10e_with_gripper prefix="''"/>
-  <xacro:property name="width" value="0.01" />
+  <!-- add a cylinder to the world for interaction -->
+  <!-- <xacro:property name="width" value="0.01" />
   <xacro:property name="bodylen" value="0.05" />
   <link name="cylinder_link">
@@ -28,5 +21,4 @@
               <cylinder radius="${width}" length="${bodylen}"/>
           </geometry>
-          <material name="blue"/>
       </visual>
       <collision>
@@ -40,4 +32,4 @@
       <child link="cylinder_link"/>
       <origin xyz="0.8 0 0.8" rpy="0 0 0"/>
-  </joint>
+  </joint> -->
 </robot>
