Commit message: updated to working state

File: urdf/ur10e_with_gripper_ros1.urdf.xacro (robot description, xacro)
@@ -12,7 +12,19 @@
       <parent link="${prefix}flange"/>
       <child link="${prefix}robotiq_arg2f_base_link"/>
-  </joint>
+    </joint>
+    <gazebo>
+      <plugin name="ros_control" filename="libgazebo_ros_control.so">
+        <robotNamespace>/</robotNamespace>
+        <robotSimType>gazebo_ros_control/DefaultRobotHWSim</robotSimType>
+      </plugin>
+    </gazebo>
   </xacro:macro>
   <xacro:ur10e_with_gripper prefix="''"/>
+  <link name="world"/>
+  <joint name="world_joint" type="fixed">
+    <parent link="world"/>
+    <child link="base_link"/>
+    <origin xyz="0 0 0" rpy="0 0 0"/>
+  </joint>
   <!-- add a cylinder to the world for interaction -->
   <!-- <xacro:property name="width" value="0.01" />
@@ -35,7 +47,3 @@
       <origin xyz="0.8 0 0.8" rpy="0 0 0"/>
   </joint> -->
-  <gazebo>
-    <plugin name="gazebo_ros_control" filename="libgazebo_ros_control.so" />
-    <RobotNamespace>/Orangejuice</RobotNamespace>
-  </gazebo>
 </robot>
